File: pcb_gateway/Gateway.kicad_pcb (KiCad board)
At the start: 2 copper layers, 65 x 56 mm, 41 parts, among them J1 RPi_GPIO, J10 CONN_01X02, J2 CONN_FTDI, J3 JPR_VIN, J4 JPR_MCU_TX, J5 JPR_MCU_RX, J6 CONN_BREAKOUT, J7 ANT-UFL, J8 ANT-SMA, J9 ANT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

Commit message: no message
Parts:
- moved C3 1.93 mm to (172.3, 79.7), turned to 270 degrees
- moved C7 0.78 mm to (146.0, 90.3)
- moved C8 0.51 mm to (159.6, 90.3)
- moved X1 0.32 mm to (155.3, 93.6)
Routing:
- net GND: track 453.7 -> 452.6 mm, vias 106 -> 103
- net Net-(C7-Pad2): track 9.67 -> 10.4 mm
